File: GlitchStorm3.kicad_pcb (KiCad board)
At the start: 2 copper layers, 99.8 x 80 mm, 60 parts, among them J1 PHONES, J2 LINE OUT, J3 DC 9V, SW1 TSL-A064, SW2 TSL-A064, SW3 TSL-A064, U2 MCP6002, U3 LM386

Commit message: GlitchStorm v3: bench test results, button relabel, mill marks, test sketch fixes
- docs: Test Procedure v3.0 filled in through section 5 (power, rails, bias,
  controls, audio) with notes; Build Notes: measured heights (button cap ~2 mm
  proud, no taller button needed) and the v3.1 change list
- board: button silkscreen BTN 1 / BTN 3 / BTN 2 (left to right); the centre
  button (BTN 3, D3) is MODE in the current firmware; user label moves
- enclosure: Othermill marking SVG (1590BB face, hole outlines + 1 mm centre
  marks), checked against the v3.0 board; README mill notes
- firmware/GS3_HWTest: MODE on the centre button (D3); double ADC reads and
  tone() hysteresis (fixes unstable low notes caused by the test sketch)

Co-Authored-By: Claude Opus 5.5 <noreply@anthropic.com>
Other:
- board text added: "BTN 3"
Changed lines of the file:
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@@
 		)
 		(fp_text user "${REFERENCE}"
-			(at 1.25 0 0)
+			(at -3.5 1.5 0)
 			(layer "F.Fab")
 			(effects
@@
 		(tags "push button round 12mm tact DAIER TSL-A064 KS01Q01")
 		(property "Reference" "SW1"
-			(at 0 7.6 180)
+			(at 5.5 5.25 180)
 			(layer "B.SilkS")
 			(effects
@@
 	)
 	(gr_text "BTN 2"
-		(at 139 127.2 0)
+		(at 134.25 131.25 0)
+		(layer "B.SilkS")
+		(effects
+			(font
+				(size 1 1)
+				(thickness 0.2)
+				(bold yes)
+			)
+			(justify mirror)
+		)
+	)
+	(gr_text "BTN 3"
+		(at 149.25 131.25 0)
 		(layer "B.SilkS")
 		(effects
@@
 	)
 	(gr_text "BTN 1"
-		(at 161 127.2 0)
+		(at 165.5 131 0)
 		(layer "B.SilkS")
 		(effects
