File: GlitchStorm3.kicad_sch (KiCad schematic)
At the start: 55 parts, among them J1 PHONES, J2 LINE OUT, J3 DC 9V, SW1 TSL-A064, SW2 TSL-A064, SW3 TSL-A064, U2 MCP6002, U3 LM386

Commit message: GlitchStorm v3: bench test results, button relabel, mill marks, test sketch fixes
- docs: Test Procedure v3.0 filled in through section 5 (power, rails, bias,
  controls, audio) with notes; Build Notes: measured heights (button cap ~2 mm
  proud, no taller button needed) and the v3.1 change list
- board: button silkscreen BTN 1 / BTN 3 / BTN 2 (left to right); the centre
  button (BTN 3, D3) is MODE in the current firmware; user label moves
- enclosure: Othermill marking SVG (1590BB face, hole outlines + 1 mm centre
  marks), checked against the v3.0 board; README mill notes
- firmware/GS3_HWTest: MODE on the centre button (D3); double ADC reads and
  tone() hysteresis (fixes unstable low notes caused by the test sketch)

Co-Authored-By: Claude Opus 5.5 <noreply@anthropic.com>
Other:
- moved on the sheet: C10, C11, C12, C13, C14, C15, C16, C17, C18, C19, C5, C6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
